File: Proto Board RF v2-0.kicad_pcb (KiCad board)
At the start: 2 copper layers, 122 parts, among them J1 BNC_out, J2 BNC_in, J3 SMA_vertical_out, J4 SMA_vertical_in, J5 SMA_edge_out, J6 SMA_edge_in, Q1 Q_NPN_BCE, Q2 Q_NPN_BCE, Q3 Q_NPN_BCE, Q4 Q_NPN_BCE

Commit message: Creat un test pad de 6x6 mm
Parts:
- removed Q1, Q2, Q3, Q4: Q_NPN_BCE, Package_TO_SOT_SMD:SOT-23
- removed TP1, TP10, TP11, TP12: C, TestPoint:TestPoint_Pad_4.0x4.0mm
- removed TP13, TP14, TP15, TP2: B, TestPoint:TestPoint_Pad_4.0x4.0mm
- removed TP16, TP17, TP18, TP5: E, TestPoint:TestPoint_Pad_4.0x4.0mm
Connections:
- TP19 pad 1: (no net) -> unconnected-(TP19-Pad1)
- TP20 pad 1: (no net) -> unconnected-(TP20-Pad1)
- TP21 pad 1: (no net) -> unconnected-(TP21-Pad1)
- TP22 pad 1: (no net) -> unconnected-(TP22-Pad1)
- TP23 pad 1: (no net) -> unconnected-(TP23-Pad1)
- TP24 pad 1: (no net) -> unconnected-(TP24-Pad1)
- TP25 pad 1: (no net) -> unconnected-(TP25-Pad1)
- TP26 pad 1: (no net) -> unconnected-(TP26-Pad1)
- TP27 pad 1: (no net) -> unconnected-(TP27-Pad1)
- TP28 pad 1: (no net) -> unconnected-(TP28-Pad1)
- TP29 pad 1: (no net) -> unconnected-(TP29-Pad1)
- TP30 pad 1: (no net) -> unconnected-(TP30-Pad1)
- TP31 pad 1: (no net) -> unconnected-(TP31-Pad1)
- TP32 pad 1: (no net) -> unconnected-(TP32-Pad1)
- TP33 pad 1: (no net) -> unconnected-(TP33-Pad1)
- TP34 pad 1: (no net) -> unconnected-(TP34-Pad1)
- TP35 pad 1: (no net) -> unconnected-(TP35-Pad1)
- TP36 pad 1: (no net) -> unconnected-(TP36-Pad1)
- TP37 pad 1: (no net) -> unconnected-(TP37-Pad1)
- TP38 pad 1: (no net) -> unconnected-(TP38-Pad1)
- TP39 pad 1: (no net) -> unconnected-(TP39-Pad1)
- TP40 pad 1: (no net) -> unconnected-(TP40-Pad1)
- TP41 pad 1: (no net) -> unconnected-(TP41-Pad1)
- TP42 pad 1: (no net) -> unconnected-(TP42-Pad1)
- TP43 pad 1: (no net) -> unconnected-(TP43-Pad1)
- TP44 pad 1: (no net) -> unconnected-(TP44-Pad1)
- TP45 pad 1: (no net) -> unconnected-(TP45-Pad1)
- TP46 pad 1: (no net) -> unconnected-(TP46-Pad1)
- TP47 pad 1: (no net) -> unconnected-(TP47-Pad1)
- TP48 pad 1: (no net) -> unconnected-(TP48-Pad1)
- TP49 pad 1: (no net) -> unconnected-(TP49-Pad1)
- TP50 pad 1: (no net) -> unconnected-(TP50-Pad1)
- TP51 pad 1: (no net) -> unconnected-(TP51-Pad1)
- TP52 pad 1: (no net) -> unconnected-(TP52-Pad1)
- TP53 pad 1: (no net) -> unconnected-(TP53-Pad1)
- TP54 pad 1: (no net) -> unconnected-(TP54-Pad1)
- TP55 pad 1: (no net) -> unconnected-(TP55-Pad1)
- TP56 pad 1: (no net) -> unconnected-(TP56-Pad1)
- TP57 pad 1: (no net) -> unconnected-(TP57-Pad1)
- TP58 pad 1: (no net) -> unconnected-(TP58-Pad1)
- TP59 pad 1: (no net) -> unconnected-(TP59-Pad1)
- TP60 pad 1: (no net) -> unconnected-(TP60-Pad1)
- TP61 pad 1: (no net) -> unconnected-(TP61-Pad1)
- TP62 pad 1: (no net) -> unconnected-(TP62-Pad1)
- TP63 pad 1: (no net) -> unconnected-(TP63-Pad1)
- TP64 pad 1: (no net) -> unconnected-(TP64-Pad1)
- TP65 pad 1: (no net) -> unconnected-(TP65-Pad1)
- TP66 pad 1: (no net) -> unconnected-(TP66-Pad1)
- TP67 pad 1: (no net) -> unconnected-(TP67-Pad1)
- TP68 pad 1: (no net) -> unconnected-(TP68-Pad1)
- TP69 pad 1: (no net) -> unconnected-(TP69-Pad1)
- TP70 pad 1: (no net) -> unconnected-(TP70-Pad1)
- TP71 pad 1: (no net) -> unconnected-(TP71-Pad1)
- TP72 pad 1: (no net) -> unconnected-(TP72-Pad1)
- TP73 pad 1: (no net) -> unconnected-(TP73-Pad1)
- TP74 pad 1: (no net) -> unconnected-(TP74-Pad1)
- TP75 pad 1: (no net) -> unconnected-(TP75-Pad1)
- TP76 pad 1: (no net) -> unconnected-(TP76-Pad1)
- TP77 pad 1: (no net) -> unconnected-(TP77-Pad1)
- TP78 pad 1: (no net) -> unconnected-(TP78-Pad1)
- TP79 pad 1: (no net) -> unconnected-(TP79-Pad1)
- TP80 pad 1: (no net) -> unconnected-(TP80-Pad1)
- TP81 pad 1: (no net) -> unconnected-(TP81-Pad1)
- TP82 pad 1: (no net) -> unconnected-(TP82-Pad1)
