File: Proto Board RF v2-0.kicad_sch (KiCad schematic)
At the start: 122 parts, among them J1 BNC_out, J2 BNC_in, J3 SMA_vertical_out, J4 SMA_vertical_in, J5 SMA_edge_out, J6 SMA_edge_in, Q1 Q_NPN_BCE, Q2 Q_NPN_BCE, Q3 Q_NPN_BCE, Q4 Q_NPN_BCE

Commit message: Creat un test pad de 6x6 mm
Parts:
- removed Q1, Q2, Q3, Q4: Q_NPN_BCE, Package_TO_SOT_SMD:SOT-23, symbol Device:Q_NPN_BCE
- removed TP1, TP10, TP11, TP12: C, TestPoint:TestPoint_Pad_4.0x4.0mm, symbol Connector:TestPoint_Alt
- removed TP13, TP14, TP15, TP2: B, TestPoint:TestPoint_Pad_4.0x4.0mm, symbol Connector:TestPoint_Alt
- removed TP16, TP17, TP18, TP5: E, TestPoint:TestPoint_Pad_4.0x4.0mm, symbol Connector:TestPoint_Alt
- gave numbers to parts that had none: 13
